Commit message: Added ball

File: urdf/ball.urdf (robot description, URDF)
Before this commit: robot sphere_robot, 1 links, 0 joints
Links:
- link ball_link: geometry collision sphere radius=0.0325; visual sphere radius=0.065

Commit message: Fixed ball

File: urdf/ball.urdf (robot description, URDF)
Before this commit: robot sphere_robot, 1 links, 0 joints
Links:
- link ball_link: geometry collision sphere radius=0.0325; visual sphere radius=0.0325
