Commit message: Fixed xacro

File: urdf/robot.xacro (robot description, xacro)
@@ -13,5 +13,5 @@
     <origin xyz="0 0 0" rpy="0 0 0"/>
     <geometry>
-      <mesh filename="file://$(find robot_description)/meshes/base_link.stl" scale="0.001 0.001 0.001"/>
+      <mesh filename="file://$(find yasarobo2025_26)/meshes/base_link.stl" scale="0.001 0.001 0.001"/>
     </geometry>
     <material name="steel_satin"/>
@@ -20,5 +20,5 @@
     <origin xyz="0 0 0" rpy="0 0 0"/>
     <geometry>
-      <mesh filename="file://$(find robot_description)/meshes/base_link.stl" scale="0.001 0.001 0.001"/>
+      <mesh filename="file://$(find yasarobo2025_26)/meshes/base_link.stl" scale="0.001 0.001 0.001"/>
     </geometry>
   </collision>
@@ -33,5 +33,5 @@
     <origin xyz="-0.007243 -0.081923 0.003" rpy="0 0 0"/>
     <geometry>
-      <mesh filename="file://$(find robot_description)/meshes/alm_1_v4_1.stl" scale="0.001 0.001 0.001"/>
+      <mesh filename="file://$(find yasarobo2025_26)/meshes/alm_1_v4_1.stl" scale="0.001 0.001 0.001"/>
     </geometry>
     <material name="aluminum_satin"/>
@@ -40,5 +40,5 @@
     <origin xyz="-0.007243 -0.081923 0.003" rpy="0 0 0"/>
     <geometry>
-      <mesh filename="file://$(find robot_description)/meshes/alm_1_v4_1.stl" scale="0.001 0.001 0.001"/>
+      <mesh filename="file://$(find yasarobo2025_26)/meshes/alm_1_v4_1.stl" scale="0.001 0.001 0.001"/>
     </geometry>
   </collision>
@@ -53,5 +53,5 @@
     <origin xyz="-0.020233 -0.089423 0.013" rpy="0 0 0"/>
     <geometry>
-      <mesh filename="file://$(find robot_description)/meshes/chassis_unit_v18_1.stl" scale="0.001 0.001 0.001"/>
+      <mesh filename="file://$(find yasarobo2025_26)/meshes/chassis_unit_v18_1.stl" scale="0.001 0.001 0.001"/>
     </geometry>
     <material name="steel_satin"/>
@@ -60,5 +60,5 @@
     <origin xyz="-0.020233 -0.089423 0.013" rpy="0 0 0"/>
     <geometry>
-      <mesh filename="file://$(find robot_description)/meshes/chassis_unit_v18_1.stl" scale="0.001 0.001 0.001"/>
+      <mesh filename="file://$(find yasarobo2025_26)/meshes/chassis_unit_v18_1.stl" scale="0.001 0.001 0.001"/>
     </geometry>
   </collision>
@@ -73,5 +73,5 @@
     <origin xyz="-0.072195 -0.059423 0.013" rpy="0 0 0"/>
     <geometry>
-      <mesh filename="file://$(find robot_description)/meshes/alm_with_lidar_v6_1.stl" scale="0.001 0.001 0.001"/>
+      <mesh filename="file://$(find yasarobo2025_26)/meshes/alm_with_lidar_v6_1.stl" scale="0.001 0.001 0.001"/>
     </geometry>
     <material name="aluminum_satin"/>
@@ -80,5 +80,5 @@
     <origin xyz="-0.072195 -0.059423 0.013" rpy="0 0 0"/>
     <geometry>
-      <mesh filename="file://$(find robot_description)/meshes/alm_with_lidar_v6_1.stl" scale="0.001 0.001 0.001"/>
+      <mesh filename="file://$(find yasarobo2025_26)/meshes/alm_with_lidar_v6_1.stl" scale="0.001 0.001 0.001"/>
     </geometry>
   </collision>
@@ -93,5 +93,5 @@
     <origin xyz="-0.072195 0.060577 0.013" rpy="0 0 0"/>
     <geometry>
-      <mesh filename="file://$(find robot_description)/meshes/chassis_unit_v18_2.stl" scale="0.001 0.001 0.001"/>
+      <mesh filename="file://$(find yasarobo2025_26)/meshes/chassis_unit_v18_2.stl" scale="0.001 0.001 0.001"/>
     </geometry>
     <material name="steel_satin"/>
@@ -100,5 +100,5 @@
     <origin xyz="-0.072195 0.060577 0.013" rpy="0 0 0"/>
     <geometry>
-      <mesh filename="file://$(find robot_description)/meshes/chassis_unit_v18_2.stl" scale="0.001 0.001 0.001"/>
+      <mesh filename="file://$(find yasarobo2025_26)/meshes/chassis_unit_v18_2.stl" scale="0.001 0.001 0.001"/>
     </geometry>
   </collision>
@@ -113,5 +113,5 @@
     <origin xyz="-0.020233 0.090577 0.013" rpy="0 0 0"/>
     <geometry>
-      <mesh filename="file://$(find robot_description)/meshes/alm_1_v4_2.stl" scale="0.001 0.001 0.001"/>
+      <mesh filename="file://$(find yasarobo2025_26)/meshes/alm_1_v4_2.stl" scale="0.001 0.001 0.001"/>
     </geometry>
     <material name="aluminum_satin"/>
@@ -120,5 +120,5 @@
     <origin xyz="-0.020233 0.090577 0.013" rpy="0 0 0"/>
     <geometry>
-      <mesh filename="file://$(find robot_description)/meshes/alm_1_v4_2.stl" scale="0.001 0.001 0.001"/>
+      <mesh filename="file://$(find yasarobo2025_26)/meshes/alm_1_v4_2.stl" scale="0.001 0.001 0.001"/>
     </geometry>
   </collision>
@@ -133,5 +133,5 @@
     <origin xyz="0.08369 -0.029423 0.013" rpy="0 0 0"/>
     <geometry>
-      <mesh filename="file://$(find robot_description)/meshes/chassis_unit_v18_3.stl" scale="0.001 0.001 0.001"/>
+      <mesh filename="file://$(find yasarobo2025_26)/meshes/chassis_unit_v18_3.stl" scale="0.001 0.001 0.001"/>
     </geometry>
     <material name="steel_satin"/>
@@ -140,5 +140,5 @@
     <origin xyz="0.08369 -0.029423 0.013" rpy="0 0 0"/>
     <geometry>
-      <mesh filename="file://$(find robot_description)/meshes/chassis_unit_v18_3.stl" scale="0.001 0.001 0.001"/>
+      <mesh filename="file://$(find yasarobo2025_26)/meshes/chassis_unit_v18_3.stl" scale="0.001 0.001 0.001"/>
     </geometry>
   </collision>
@@ -153,5 +153,5 @@
     <origin xyz="-0.072195 0.023977 0.013" rpy="0 0 0"/>
     <geometry>
-      <mesh filename="file://$(find robot_description)/meshes/LD19_with_mounter_v17_1.stl" scale="0.001 0.001 0.001"/>
+      <mesh filename="file://$(find yasarobo2025_26)/meshes/LD19_with_mounter_v17_1.stl" scale="0.001 0.001 0.001"/>
     </geometry>
     <material name="steel_satin"/>
@@ -160,5 +160,5 @@
     <origin xyz="-0.072195 0.023977 0.013" rpy="0 0 0"/>
     <geometry>
-      <mesh filename="file://$(find robot_description)/meshes/LD19_with_mounter_v17_1.stl" scale="0.001 0.001 0.001"/>
+      <mesh filename="file://$(find yasarobo2025_26)/meshes/LD19_with_mounter_v17_1.stl" scale="0.001 0.001 0.001"/>
     </geometry>
   </collision>
@@ -173,5 +173,5 @@
     <origin xyz="0.044719 0.053077 0.013" rpy="0 0 0"/>
     <geometry>
-      <mesh filename="file://$(find robot_description)/meshes/fun_adapter_v2_1.stl" scale="0.001 0.001 0.001"/>
+      <mesh filename="file://$(find yasarobo2025_26)/meshes/fun_adapter_v2_1.stl" scale="0.001 0.001 0.001"/>
     </geometry>
     <material name="steel_satin"/>
@@ -180,5 +180,5 @@
     <origin xyz="0.044719 0.053077 0.013" rpy="0 0 0"/>
     <geometry>
-      <mesh filename="file://$(find robot_description)/meshes/fun_adapter_v2_1.stl" scale="0.001 0.001 0.001"/>
+      <mesh filename="file://$(find yasarobo2025_26)/meshes/fun_adapter_v2_1.stl" scale="0.001 0.001 0.001"/>
     </geometry>
   </collision>
@@ -193,5 +193,5 @@
     <origin xyz="0.065593 0.061233 0.016" rpy="0 0 0"/>
     <geometry>
-      <mesh filename="file://$(find robot_description)/meshes/fun_v13_1.stl" scale="0.001 0.001 0.001"/>
+      <mesh filename="file://$(find yasarobo2025_26)/meshes/fun_v13_1.stl" scale="0.001 0.001 0.001"/>
     </geometry>
     <material name="steel_satin"/>
@@ -200,5 +200,5 @@
     <origin xyz="0.065593 0.061233 0.016" rpy="0 0 0"/>
     <geometry>
-      <mesh filename="file://$(find robot_description)/meshes/fun_v13_1.stl" scale="0.001 0.001 0.001"/>
+      <mesh filename="file://$(find yasarobo2025_26)/meshes/fun_v13_1.stl" scale="0.001 0.001 0.001"/>
     </geometry>
   </collision>

Commit message: Fixed urdf

File: urdf/robot.xacro (robot description, xacro)
@@ -234,9 +234,4 @@
   <child link="chassis_unit_v18_3"/>
 </joint>
-<joint name="Rigid 9" type="fixed">
-  <origin xyz="0.0 -0.0834 0.0" rpy="0 0 0"/>
-  <parent link="alm_with_lidar_v6_1"/>
-  <child link="LD19_with_mounter_v17_1"/>
-</joint>
 <joint name="Rigid 10" type="fixed">
   <origin xyz="-0.064952 0.0375 0.0" rpy="0 0 0"/>
@@ -248,4 +243,9 @@
   <parent link="fun_adapter_v2_1"/>
   <child link="fun_v13_1"/>
+</joint>
+<joint name="Rigid 13" type="fixed">
+  <origin xyz="0.0 -0.0834 0.0" rpy="0 0 0"/>
+  <parent link="alm_with_lidar_v6_1"/>
+  <child link="LD19_with_mounter_v17_1"/>
 </joint>
   <link name="base_footprint">

Commit message: test

File: urdf/robot.xacro (robot description, xacro)
@@ -271,10 +271,10 @@
     <parent link="LD19_with_mounter_v17_1"/>
     <child  link="ldlidar_base"/>
-    <origin xyz="0.033 0.013 -0.05" rpy="0 0 0"/>
+    <origin xyz="0.0 0.0 -0.1" rpy="0 0 0"/>
   </joint>
   <gazebo reference="ldlidar_base">
     <sensor type="gpu_lidar" name="lidar_sensor">
       <ignition_frame_id>ldlidar_base</ignition_frame_id>
-      <topic>/ldlidar_node/scan</topic>
+      <topic>/scan_back</topic>
       <alwaysOn>1</alwaysOn>
       <visualize>true</visualize>

Commit message: urdf change

File: urdf/robot.xacro (robot description, xacro)
@@ -269,5 +269,5 @@
   <link name="ldlidar_base"/>
   <joint name="lidar_joint" type="fixed">
-    <parent link="LD19_with_mounter_v17_1"/>
+    <parent link="base_link"/>
     <child  link="ldlidar_base"/>
     <origin xyz="0.0 0.0 -0.1" rpy="0 0 0"/>

Commit message: test

File: urdf/robot.xacro (robot description, xacro)
@@ -267,13 +267,13 @@
   </joint>
    <!-- LiDAR -->
-  <link name="ldlidar_base"/>
+  <link name="lidar_base"/>
   <joint name="lidar_joint" type="fixed">
     <parent link="base_link"/>
-    <child  link="ldlidar_base"/>
-    <origin xyz="0.0 0.0 -0.1" rpy="0 0 0"/>
+    <child  link="lidar_base"/>
+    <origin xyz="0.0 0.0 -0.1" rpy="1.57 0 0"/>
   </joint>
-  <gazebo reference="ldlidar_base">
+  <gazebo reference="lidar_base">
     <sensor type="gpu_lidar" name="lidar_sensor">
-      <ignition_frame_id>ldlidar_base</ignition_frame_id>
+      <ignition_frame_id>lidar_base</ignition_frame_id>
       <topic>/scan_back</topic>
       <alwaysOn>1</alwaysOn>

Commit message: test

File: urdf/robot.xacro (robot description, xacro)
@@ -271,5 +271,5 @@
     <parent link="base_link"/>
     <child  link="lidar_base"/>
-    <origin xyz="0.0 0.0 -0.1" rpy="1.57 0 0"/>
+    <origin xyz="0.0 0.0 -0.1" rpy="3.14 0 0.785"/>
   </joint>
   <gazebo reference="lidar_base">

Commit message: test

File: urdf/robot.xacro (robot description, xacro)
@@ -271,5 +271,5 @@
     <parent link="base_link"/>
     <child  link="lidar_base"/>
-    <origin xyz="0.0 0.0 -0.1" rpy="3.14 0 0.785"/>
+    <origin xyz="0.0 0.0 -0.1" rpy="3.14 0 0"/>
   </joint>
   <gazebo reference="lidar_base">

Commit message: test

File: urdf/robot.xacro (robot description, xacro)
@@ -271,5 +271,5 @@
     <parent link="base_link"/>
     <child  link="lidar_base"/>
-    <origin xyz="0.0 0.0 -0.1" rpy="3.14 0 0"/>
+    <origin xyz="0.0 0.0 -0.1" rpy="3.14 0 1.57"/>
   </joint>
   <gazebo reference="lidar_base">

Commit message: test

File: urdf/robot.xacro (robot description, xacro)
@@ -271,5 +271,5 @@
     <parent link="base_link"/>
     <child  link="lidar_base"/>
-    <origin xyz="0.0 0.0 -0.1" rpy="3.14 0 1.57"/>
+    <origin xyz="0.0 0.0 -0.1" rpy="3.14 0 -0.785"/>
   </joint>
   <gazebo reference="lidar_base">

Commit message: urdf ok

File: urdf/robot.xacro (robot description, xacro)
@@ -271,5 +271,5 @@
     <parent link="base_link"/>
     <child  link="lidar_base"/>
-    <origin xyz="0.0 0.0 -0.1" rpy="3.14 0 -0.785"/>
+    <origin xyz="0.0 0.0 -0.1" rpy="3.14 0 -2.09333"/>
   </joint>
   <gazebo reference="lidar_base">
